Commit message: Initial Commit

File: baxter_sim_examples/models/block/model1.urdf (robot description, URDF)
Before this commit: robot block, 1 links, 0 joints
Links:
- link block: geometry collision box size=0.35 0.73 0.64; visual box size=0.35 0.73 0.64

File: baxter_sim_examples/models/block/model2.urdf (robot description, URDF)
Before this commit: robot block, 1 links, 0 joints
Links:
- link block: geometry collision box size=0.05 0.05 0.05; visual box size=0.05 0.05 0.05

File: baxter_sim_examples/models/block/model3.urdf (robot description, URDF)
Before this commit: robot block, 1 links, 0 joints
Links:
- link block: geometry collision box size=0.05 0.05 0.05; visual box size=0.05 0.05 0.05
